File: LaserCAN-Board/LaserCAN-Board.kicad_sch (KiCad schematic)
At the start: 57 parts, among them J2 TC2050-IDC-NL, Q1 Si2309CDS-T1-GE3, U1 TPS7A2033PDBVR, U10 M24C64-RMN6TP, U2 VL53L1CXV0FY1, U4 STM32F103C8Tx, U9 SN65HVD230, U9 TPS54202DDC, Y1 8MHz 12pF

Commit message: Slight part number change
Parts:
- D3: LCSC Part C72043 -> C965804
Changed lines of the file:
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@@
       (effects (font (size 1.27 1.27)) hide)
     )
-    (property "LCSC Part" "C72043" (at 217.17 252.73 0)
+    (property "LCSC Part" "C965804" (at 217.17 252.73 0)
       (effects (font (size 1.27 1.27)) hide)
     )

Commit message: Start working on Rev5
Parts:
- R9: value 4.7 100mW -> 4.7; LCSC Part C3009058 -> C491192
Connections:
- net +12V: now also J2.1; no longer J2.10, J2.9
- net GND: now also U4.3 (PC14); no longer J2.4
- net NRST: now also J2.10; no longer J2.1
- net TOF_SHUT: now also U4.45 (PB8); no longer U4.40 (PB4)
- net JTDI: now reaches J2.8
- net JTDI: now also U4.38 (PA15)
- net JTDO: now reaches U4.39 (PB3)
- net JTDO: now also J2.6
- net SWCLK renamed SWCLK/JTCK
- net SWCLK/JTCK: now also J2.4; no longer J2.6
- net SWDIO renamed SWDIO/JTMS
- no-connect marks 32 -> 29
Other:
- note added: "CRCW06034R70JNEAHP (C3009058) for pulse ALT ERJ-UP3J4R7V (C491192)"
- note added: "NOTE: Updated for Rev 5 to be TC Standard for use with TC2050-ARM2010"
- note removed: "CRCW06034R70JNEAHP for pulse"

Commit message: Slight changes
Connections:
- net +12V: now also J2.5; no longer J2.1
- net +3V3: now also J2.1
- no-connect marks 29 -> 28
Changed lines of the file:
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@@
   (no_connect (at 101.6 82.55))
   (no_connect (at 101.6 92.71))
-  (no_connect (at 93.98 210.82))
   (no_connect (at 58.42 223.52))
   (no_connect (at 123.19 208.28))
@@
     (stroke (width 0) (type default))
   )
+  (wire (pts (xy 92.71 199.39) (xy 92.71 200.66))
+    (stroke (width 0) (type default))
+  )
   (wire (pts (xy 134.62 85.09) (xy 148.59 85.09))
     (stroke (width 0) (type default))
@@
     (stroke (width 0) (type default))
   )
+  (wire (pts (xy 92.71 200.66) (xy 95.25 200.66))
+    (stroke (width 0) (type default))
+  )
   (wire (pts (xy 116.84 128.27) (xy 118.11 128.27))
     (stroke (width 0) (type default))
@@
     (stroke (width 0) (type default))
   )
+  (wire (pts (xy 83.82 210.82) (xy 95.25 210.82))
+    (stroke (width 0) (type default))
+  )
   (wire (pts (xy 78.74 77.47) (xy 78.74 80.01))
     (stroke (width 0) (type default))
@@
     (stroke (width 0) (type default))
   )
-  (wire (pts (xy 95.25 200.66) (xy 85.09 200.66))
-    (stroke (width 0) (type default))
-  )
   (wire (pts (xy 179.07 198.12) (xy 167.64 198.12))
     (stroke (width 0) (type default))
@@
     (stroke (width 0) (type default))
   )
-  (wire (pts (xy 93.98 210.82) (xy 95.25 210.82))
-    (stroke (width 0) (type default))
-  )
   (wire (pts (xy 259.08 135.89) (xy 254 135.89))
     (stroke (width 0) (type default))
@@
     (fill (type none))
   )
-  (rectangle (start 77.47 181.61) (end 187.96 271.78)
+  (rectangle (start 76.2 181.61) (end 191.77 271.78)
     (stroke (width 0) (type default))
     (fill (type none))
@@
     (effects (font (size 1.27 1.27)) (justify right bottom))
   )
+  (label "PWR_IN" (at 83.82 210.82 0) (fields_autoplaced)
+    (effects (font (size 1.27 1.27)) (justify left bottom))
+  )
   (label "BUCK_SW" (at 280.67 64.77 0) (fields_autoplaced)
     (effects (font (size 1.27 1.27)) (justify left bottom))
@@
   (label "SWDIO{slash}JTMS" (at 148.59 87.63 180) (fields_autoplaced)
     (effects (font (size 1.27 1.27)) (justify right bottom))
-  )
-  (label "PWR_IN" (at 85.09 200.66 0) (fields_autoplaced)
-    (effects (font (size 1.27 1.27)) (justify left bottom))
   )
   (label "NRST" (at 132.08 200.66 180) (fields_autoplaced)
@@
         )
       )
+    )
+  )
+  (symbol (lib_id "power:+3V3") (at 92.71 199.39 0) (unit 1)
+    (in_bom yes) (on_board yes) (dnp no)
+    (property "Reference" "#PWR0196" (at 92.71 203.2 0)
+      (effects (font (size 1.27 1.27)) hide)
+    )
+    (property "Value" "+3V3" (at 92.71 195.58 0)
+      (effects (font (size 1.27 1.27)))
+    )
+    (property "Footprint" "" (at 92.71 199.39 0)
+      (effects (font (size 1.27 1.27)) hide)
+    )
+    (property "Datasheet" "" (at 92.71 199.39 0)
+      (effects (font (size 1.27 1.27)) hide)
+    )
+    (pin "1")
+    (instances
+      (project "spiderlan-mxp"
+        (path "/2e542182-4621-486d-ae69-beec03baa0f5"
+          (reference "#PWR0196") (unit 1)
+        )
+      )
+      (project "spiderlan-baseboard"
+        (path "/30d29dde-b352-4ed5-b433-0a69e9c9f163"
+          (reference "#PWR06") (unit 1)
+        )
+      )
+      (project "LaserCAN-Board"
+        (path "/397780dc-ec79-4cd5-82ec-d7f123571087"
+          (reference "#PWR033") (unit 1)
+        )
+      )
